File: eagle/project_schematic.sch (EAGLE design)
At the start: 17 parts, among them Q1 2N3904, Q2 2N3904, Q3 2N3906

Commit message: Update design
Connections:
- net GND: now also 9V_SPKR.4
Changed lines of the file:
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@@
 <wire x1="78.74" y1="93.98" x2="78.74" y2="96.52" width="0.1524" layer="91"/>
 <junction x="78.74" y="96.52"/>
+<wire x1="78.74" y1="93.98" x2="78.74" y2="91.44" width="0.1524" layer="91"/>
+<junction x="78.74" y="93.98"/>
+<pinref part="9V_SPKR" gate="G$1" pin="4"/>
+<wire x1="78.74" y1="91.44" x2="81.28" y2="91.44" width="0.1524" layer="91"/>
 </segment>
 <segment>
